Commit message: ล่าสุด

File: install/control_rbkairos/share/control_rbkairos/urdf/rbrobout.urdf.xacro (robot description, xacro)
@@ -1 +1,66 @@
-/home/khotkangplue_p/week6_ws/build/control_rbkairos/urdf/rbrobout.urdf.xacro
+<?xml version="1.0" ?>
+<robot
+  name="rbrobout"
+  xmlns:xacro="http://wiki.ros.org/xacro">
+  <xacro:include
+    filename="$(find robotnik_description)/urdf/bases/rbrobout/rbrobout_base.urdf.xacro" />
+  <xacro:include
+    filename="$(find robotnik_sensors)/urdf/all_sensors.urdf.xacro" />
+  <!-- ARGUMENTS -->
+  <xacro:arg
+    name="namespace"
+    default="robot" />
+  <xacro:arg
+    name="prefix"
+    default="" />
+  <xacro:arg
+    name="gazebo_ignition"
+    default="false" />
+  <!-- RB-ROBOUT -->
+  <xacro:rbrobout
+    prefix="$(arg prefix)"
+    gazebo_ignition="$(arg gazebo_ignition)"
+    namespace="$(arg namespace)" />
+  <!-- IMU -->
+  <xacro:sensor_vectornav
+    frame_prefix="$(arg prefix)imu_"
+    parent="$(arg prefix)base_link"
+    node_namespace="$(arg namespace)"
+    gazebo_ignition="$(arg gazebo_ignition)">
+    <origin
+      xyz="0.3 -0.3 0.0725"
+      rpy="0 0 0" />
+  </xacro:sensor_vectornav>
+  <!-- LASERS -->
+  <xacro:sensor_sick_microscan3
+    frame_prefix="$(arg prefix)front_laser_"
+    parent="$(arg prefix)base_link"
+    node_namespace="$(arg namespace)"
+    node_name="front_laser"
+    gazebo_ignition="$(arg gazebo_ignition)">
+    <origin
+      xyz="0.8 0.366 -0.06"
+      rpy="0 0 ${1/4*pi}" />
+  </xacro:sensor_sick_microscan3>
+  <xacro:sensor_sick_microscan3
+    frame_prefix="$(arg prefix)rear_laser_"
+    parent="$(arg prefix)base_link"
+    node_namespace="$(arg namespace)"
+    node_name="rear_laser"
+    gazebo_ignition="$(arg gazebo_ignition)">
+    <origin
+      xyz="-0.8 -0.366 -0.06"
+      rpy="0 0 ${-3/4*pi}" />
+  </xacro:sensor_sick_microscan3>
+  <!-- CAMERAS -->
+  <xacro:sensor_intel_realsense_d435
+    frame_prefix="$(arg prefix)front_rgbd_camera_"
+    parent="$(arg prefix)base_link"
+    node_namespace="$(arg namespace)"
+    node_name="front_camera"
+    gazebo_ignition="$(arg gazebo_ignition)">
+    <origin
+      xyz="0.835 0 0.1555"
+      rpy="0 0 0" />
+  </xacro:sensor_intel_realsense_d435>
+</robot>
